File: Hardware/Split_keyboard/Split_keyboard.kicad_pcb (KiCad board)
At the start: 2 copper layers, 312.9 x 117 mm, 125 parts, among them SW1 SW_Push, SW10 SW_Push, SW11 SW_Push, SW12 SW_Push, SW13 SW_Push, SW14 SW_Push, SW15 SW_Push, SW16 SW_Push, SW17 SW_Push, SW18 SW_Push, SW19 SW_Push, SW2 SW_Push, SW20 SW_Push, SW21 SW_Push, SW22 SW_Push, SW23 SW_Push, SW24 SW_Push, SW25 SW_Push, SW26 SW_Push, SW27 SW_Push, SW28 SW_Push, SW29 SW_Push, SW3 SW_Push, SW30 SW_Push, SW31 SW_Push, SW32 SW_Push, SW33 SW_Push, SW34 SW_Push, SW35 SW_Push, SW36 SW_Push, SW37 SW_Push, SW38 SW_Push, SW39 SW_Push, SW4 SW_Push, SW40 SW_Push, SW41 SW_Push, SW42 SW_Push, SW43 SW_Push, SW44 SW_Push, SW45 SW_Push, SW46 SW_Push, SW47 SW_Push, SW48 SW_Push, SW49 SW_Push, SW5 SW_Push, SW50 SW_Push, SW51 SW_Push, SW52 SW_Push, SW53 SW_Push, SW54 SW_Push, SW55 SW_Push, SW56 SW_Push, SW6 SW_Push, SW7 SW_Push, SW8 SW_Push, SW9 SW_Push, U3 SuperMini nRF52840, U4 SuperMini nRF52840

Commit message: Add initial schematic and PDF documentation for split keyboard design
- Created a new schematic file for the split keyboard in KiCad format.
- Added a PDF document for the split keyboard design.
Parts:
- removed BO6, BO7: Break Off, Panelization.pretty-master:mouse-bite-5mm-slot
- removed BO8: Break off, Panelization.pretty-master:mouse-bite-5mm-slot
- added H1: MountingHole, MountingHole:MountingHole_2.2mm_M2, F.Cu at (299.7, 71.1)
- added H10: MountingHole, MountingHole:MountingHole_2.2mm_M2, F.Cu at (111.8, 68.6)
- added H11: MountingHole, MountingHole:MountingHole_2.2mm_M2, F.Cu at (218.4, 109.2)
- added H12: MountingHole, MountingHole:MountingHole_2.2mm_M2, F.Cu at (111.8, 109.2)
- added H2: MountingHole, MountingHole:MountingHole_2.2mm_M2, F.Cu at (30.5, 71.1)
- added H3: MountingHole, MountingHole:MountingHole_2.2mm_M2, F.Cu at (299.7, 111.8)
- added H4: MountingHole, MountingHole:MountingHole_2.2mm_M2, F.Cu at (30.5, 109.2)
- added H5: MountingHole, MountingHole:MountingHole_2.2mm_M2, F.Cu at (259.1, 68.6)
- added H6: MountingHole, MountingHole:MountingHole_2.2mm_M2, F.Cu at (71.1, 68.6)
- added H7: MountingHole, MountingHole:MountingHole_2.2mm_M2, F.Cu at (259.1, 106.7)
- added H8: MountingHole, MountingHole:MountingHole_2.2mm_M2, F.Cu at (71.1, 106.7)
- added H9: MountingHole, MountingHole:MountingHole_2.2mm_M2, F.Cu at (218.4, 68.6)
- moved R2 13.0 mm to (279.4, 137.2)
- moved R1 12.9 mm to (279.4, 144.8)
Routing:
- net VBAT: track 0.00 -> 199.4 mm
- net GND: track 41.2 -> 153.2 mm
- net BT_PIN: track 38.7 -> 46.3 mm
- net R1: track 423.5 -> 418.8 mm
- net C6: track 130.1 -> 131.4 mm
